File: src/Nano2UNO-Adapter-3V3.kicad_pcb (KiCad board)
At the start: 2 copper layers, 68.6 x 53.3 mm, 19 parts, among them J1 ESW-108-33-L-S, J2 ESW-110-33-L-S, J3 ESW-108-33-L-S, J4 ESW-106-33-L-S, J5 PPPC151LFBN-RC, J6 PPPC151LFBN-RC, J7 TSW-103-15-L-D, J8 PJ-102A, SW1 1825910-6, U1 R-78K5.0-0.5

Commit message: Increased the font size of the comments and dimensions.
Other:
- board text added: "REV: ${REVISION}"
- board text removed: "REV: 0.0.1"
Changed lines of the file:
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@@
   (title_block
     (title "Nano2UNO Adapter 3V3")
-    (date "2023-12-02")
+    (date "2023-12-05")
     (rev "0.0.1")
     (company "Designer: C. M. Bulliner")
@@
       (layer "B.Paste" (type "Bottom Solder Paste"))
       (layer "B.SilkS" (type "Bottom Silk Screen"))
+      (copper_finish "None")
       (dielectric_constraints no)
     )
@@
     (aux_axis_origin 105.41 134.62)
     (pcbplotparams
-      (layerselection 0x0001000_7ffffffe)
-      (plot_on_all_layers_selection 0x0020300_00000000)
+      (layerselection 0x0000100_7ffffffe)
+      (plot_on_all_layers_selection 0x0021220_00000000)
       (disableapertmacros false)
       (usegerberextensions false)
@@
     (effects (font (size 1.5 1.5) (thickness 0.225)) (justify mirror))
   )
-  (gr_text "REV: 0.0.1" (at 157.48 102.87) (layer "B.SilkS")
+  (gr_text "REV: ${REVISION}" (at 157.48 102.87) (layer "B.SilkS")
     (effects (font (size 1 1) (thickness 0.15)) (justify mirror))
   )
@@
     (effects (font (size 1.5 1.5) (thickness 0.225)))
   )
-  (gr_text "REV: 0.0.1" (at 153.67 121.92) (layer "F.SilkS")
+  (gr_text "REV: ${REVISION}" (at 153.67 121.92) (layer "F.SilkS")
     (effects (font (size 1 1) (thickness 0.15)))
   )
@@
     (effects (font (size 1.5 1.5) (thickness 0.225)))
   )
-  (gr_text "Circuit Board Specifications\n\nBoard Thickness: 1.6mm\nSubstrate Material: FR4\nCopper Layers: 2\nCopper Thickness: 1oz\nSoldermask Color: Any (Blue Suggested)\nSurface Finish: Any (HASL Lead-Free Suggested)\n\nSmallest Hole Diameter: 0.8mm\nSmallest Trace Width: 0.2mm (7.8mil)\nSmallest Trace Spacing: 0.2mm (7.8mil)\n\nDocumentation and source files can be found at https://github.com/CMB27/Nano2UNO-Adapter-3V3." (at 15.24 200.66) (layer "Cmts.User")
-    (effects (font (size 1.27 1.27) (thickness 0.15875)) (justify left bottom))
+  (gr_text "Circuit Board Specifications\n\nBoard Thickness: 1.6mm\nSubstrate Material: FR4\nCopper Layers: 2\nCopper Thickness: 1oz\nSoldermask Color: Any (Blue Suggested)\nSurface Finish: Any (HASL Lead-Free Suggested)\n\nSmallest Hole Diameter: 0.8mm\nSmallest Trace Width: 0.2mm (7.8mil)\nSmallest Trace Spacing: 0.2mm (7.8mil)\n\nDocumentation and source files can be found at\nhttps://github.com/CMB27/Nano2UNO-Adapter-3V3." (at 15.24 200.66) (layer "Cmts.User")
+    (effects (font (size 1.5 1.5) (thickness 0.15)) (justify left bottom))
   )
   (dimension (type aligned) (layer "Dwgs.User")
@@
     (height -11.43)
     (gr_text "53.34 mm" (at 93.98 107.95 90) (layer "Dwgs.User")
-      (effects (font (size 1 1) (thickness 0.15)))
+      (effects (font (size 1.5 1.5) (thickness 0.15)))
     )
     (format (prefix "") (suffix "") (units 2) (units_format 1) (precision 2))
@@
     (height 7.62)
     (gr_text "68.58 mm" (at 139.7 142.24) (layer "Dwgs.User")
-      (effects (font (size 1 1) (thickness 0.15)))
+      (effects (font (size 1.5 1.5) (thickness 0.15)))
     )
     (format (prefix "") (suffix "") (units 2) (units_format 1) (precision 2))
