File: src/Nano2UNO-Adapter-3V3.kicad_pcb (KiCad board)
At the start: 2 copper layers, 68.6 x 53.3 mm, 19 parts, among them J1 ESW-108-33-L-S, J2 ESW-110-33-L-S, J3 ESW-108-33-L-S, J4 ESW-106-33-L-S, J5 PPPC151LFBN-RC, J6 PPPC151LFBN-RC, J7 TSW-103-15-L-D, J8 PJ-102A, SW1 1825910-6, U1 R-78K5.0-0.5

Commit message: Added additional part metadata to the schematic. Changed RST to RESET on one of the schematic symbols. Changed the revision from 1.0.0 to 1.0.1.
Parts:
- removed REF**: OSHW-Logo_11.4x12mm_SilkScreen, Symbol:OSHW-Logo_11.4x12mm_SilkScreen
- removed REF**: KiCad-Logo2_5mm_SilkScreen, Symbol:KiCad-Logo2_5mm_SilkScreen
